Commit message: update outpost and navigation config

File: src/torosamy_navigation/torosamy_navigation_server/torosamy_navigation_server_launcher/urdf/torosamy_hearvy_pancake/robot.urdf.xacro (robot description, xacro)
@@ -8,6 +8,12 @@
         <link name="livox_frame">
         </link>
+<!--
         <joint name="livox_joint" type="fixed">
             <origin xyz="0.0372 0 0.60" rpy="3.1415926 0 0" />
+            <parent link="base_link"/>
+            <child link="livox_frame"/>
+        </joint> -->
+        <joint name="livox_joint" type="fixed">
+            <origin xyz="0.0 0.045 0.49" rpy="0 0 0"/>
             <parent link="base_link"/>
             <child link="livox_frame"/>
