Commit message: try to add reality build map package

File: src/torosamy_navigation/torosamy_navigation_server/torosamy_navigation_map_builder/urdf/torosamy_hearvy_pancake/robot.urdf.xacro (robot description, xacro)
@@ -8,15 +8,14 @@
         <link name="livox_frame">
         </link>
-<!--
         <joint name="livox_joint" type="fixed">
             <origin xyz="0.0372 0 0.659" rpy="0 0 0" />
             <parent link="base_link"/>
             <child link="livox_frame"/>
-        </joint> -->
-        <joint name="livox_joint" type="fixed">
+        </joint>
+        <!-- <joint name="livox_joint" type="fixed">
             <origin xyz="0.0 0.045 0.49" rpy="0 0 0"/>
             <parent link="base_link"/>
             <child link="livox_frame"/>
-        </joint>
+        </joint> -->
     </xacro:macro>
     <xacro:base_xacro/>

File: src/torosamy_navigation/torosamy_navigation_server/torosamy_navigation_map_builder/urdf/torosamy_little_pancake/robot.urdf.xacro (robot description, xacro)
@@ -8,12 +8,6 @@
         <link name="livox_frame">
         </link>
-<!--
         <joint name="livox_joint" type="fixed">
-            <origin xyz="0.0372 0 0.659" rpy="0 0 0" />
-            <parent link="base_link"/>
-            <child link="livox_frame"/>
-        </joint> -->
-        <joint name="livox_joint" type="fixed">
-            <origin xyz="0.0 0.045 0.49" rpy="0 0 0"/>
+            <origin xyz="-0.211 0 0.28535" rpy="3.1415926 0 0" />
             <parent link="base_link"/>
             <child link="livox_frame"/>
